File: Electronics/source/separate_pcbs/libre-MiG MCU/libre-MiG MCU.kicad_sch (KiCad schematic)
At the start: 48 parts, among them J1 Conn_01x05, J16 Conn_01x02, J2 Conn_01x03, J3 Conn_01x03, J4 Conn_01x05, J6 Conn_01x20, J7 Conn_01x20, SW10 SW_Push, SW11 SW_Push, SW12 SW_Push, SW13 SW_Push, SW14 SW_Coded, SW4 SW_Push, SW5 SW_SPDT, SW6 SW_SPDT, SW7 SW_SPDT, SW8 SW_Push, SW9 SW_Push, U1 STM32F030C8Tx, U4 FT231XS, U5 ADP122AUJZ-3.3-R7, Y1 ABL-32.000MHZ-B2

Commit message: started layout and finished board shapes
Parts:
- J4: footprint Connector_JST:JST_PH_S5B-PH-K_1x05_P2.00mm_Horizontal -> Connector_JST:JST_PH_B5B-PH-K_1x05_P2.00mm_Vertical
Changed lines of the file:
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@@
     (property "Reference" "J4" (id 0) (at 33.02 81.28 0))
     (property "Value" "Conn_01x05" (id 1) (at 33.02 83.82 0))
-    (property "Footprint" "Connector_JST:JST_PH_S5B-PH-K_1x05_P2.00mm_Horizontal" (id 2) (at 33.02 92.71 0)
+    (property "Footprint" "Connector_JST:JST_PH_B5B-PH-K_1x05_P2.00mm_Vertical" (id 2) (at 33.02 92.71 0)
       (effects (font (size 1.27 1.27)) hide)
     )
